Commit message: Changed urdf link for lidar

File: jetbot_mirea_description/urdf/jetbot_mirea.urdf.xacro (robot description, xacro)
@@ -1,15 +1,4 @@
 <?xml version="1.0"?>
 <robot xmlns:xacro="http://www.ros.org/wiki/xacro" name="jetbot_mirea">
-    <!--
-    TODO:
-    ✅1. Подключение модели камеры Intel Realsense
-    2. Починить отсутствия СК колес
-    3. Привязать Rplidar A2
-    4. Проверить привязку к реальному роботу
-    5. Запилить работу модели с Gazebo
-    6. Починить, что сбиваются преобразования систем координат
-    7. ???
-    ✅8. Разобраться, что за файлики *.rviz
-        -->
     <xacro:arg name="use_nominal_extrinsics" default="false"/>
     <xacro:arg name="add_plug" default="false" />
@@ -77,7 +66,7 @@
             </geometry>
         </collision>
-        <!-- <xacro:inertial_cylinder mass="0.001" length="0.029" radius="0.032">
+        <xacro:inertial_cylinder mass="0.001" length="0.029" radius="0.032">
             <origin xyz="0.0 -0.06 -0.005" rpy="0.0 0.0 0.0"/>
-        </xacro:inertial_cylinder> -->
+        </xacro:inertial_cylinder>
     </link>
     <joint name="wheel_right_joint" type="continuous">
@@ -97,5 +86,5 @@
         </visual>
         <collision>
-            <origin xyz="0 0.06 -0.005" rpy="1.57 0 0"/>
+            <origin xyz="0 0 0" rpy="0 0 0"/>
             <geometry>
                 <cylinder length="0.029" radius="0.032"/>
@@ -231,25 +220,25 @@
         </xacro:inertial_box>
     </link>
-  <joint name="rplidar_joint" topic_ns="scan" type="fixed">
-    <parent link="base_link"/>
-    <child link="rplidar_link"/>
-    <origin xyz="0.087 0.0 -0.003" rpy="3.14 0.0 2.3562"/>
-  </joint>
-  <link name="rplidar_link">
-    <visual>
-        <origin xyz="0.0 0.0 -0.023" rpy="1.5708 0 0.7854"/>
-            <!--<geometry>
-                <cylinder length="0.038" radius="0.036"/>
-            </geometry>-->
-        <geometry>
-            <!--<cylinder length="0.038" radius="0.036"/>-->
-            <mesh filename="package://jetbot_mirea_description/meshes/rplidar.dae" scale="0.001 0.001 0.001"/>
-        </geometry>
-        <material name="black"/>
-    </visual>
-        <collision>
-            <origin xyz="0.0 0.0 0.0" rpy="3.14 0 0"/>
-            <geometry>
-                <cylinder length="0.038" radius="0.036"/>
+    <joint name="rplidar_joint" topic_ns="scan" type="fixed">
+        <parent link="base_link"/>
+        <child link="rplidar_link"/>
+        <origin xyz="0.087 0.0 -0.003" rpy="0 0.0 2.3562"/>
+    </joint>
+    <link name="rplidar_link">
+        <visual>
+            <origin xyz="0.0 0.0 -0.023" rpy="1.5708 0 0.7854"/>
+                <!--<geometry>
+                    <cylinder length="0.038" radius="0.036"/>
+                </geometry>-->
+            <geometry>
+                <!--<cylinder length="0.038" radius="0.036"/>-->
+                <mesh filename="package://jetbot_mirea_description/meshes/rplidar.dae" scale="0.001 0.001 0.001"/>
+            </geometry>
+            <material name="black"/>
+        </visual>
+        <collision>
+            <origin xyz="0.0 0.0 -0.03" rpy="3.14 0 0"/>
+            <geometry>
+                <cylinder length="0.076" radius="0.042"/>
             </geometry>
         </collision>
