Commit message: Hot fix

File: jetbot_mirea_description/urdf/jetbot_mirea_detalied.urdf.xacro (robot description, xacro)
@@ -47,9 +47,4 @@
     </joint>
     <link name="wheel_left_link">
-        <inertial>
-            <mass value="${wheel_mass}"/>
-            <origin xyz="0 0 0"/>
-            <inertia ixx="0.012411765597" ixy="-0.000711733678" ixz="0.00050272983" iyy="0.015218160428" iyz="-0.000004273467" izz="0.011763977943"/>
-        </inertial>
         <visual>
             <origin xyz="0 0 0" rpy="0 0 0"/>
@@ -66,6 +61,6 @@
             </geometry>
         </collision>
-        <xacro:inertial_cylinder mass="0.001" length="0.029" radius="0.032">
-            <origin xyz="0.0 -0.06 -0.005" rpy="0.0 0.0 0.0"/>
+        <xacro:inertial_cylinder mass="${wheel_mass}" length="0.029" radius="0.032">
+            <origin xyz="0 0 0" rpy="0 0 0"/>
         </xacro:inertial_cylinder>
     </link>
