Commit message: Added PID fix

File: jetbot_mirea_description/urdf/jetbot_mirea_simple_gazebo_real.urdf.xacro (robot description, xacro)
@@ -39,10 +39,10 @@
     <xacro:include filename="$(find jetbot_mirea_description)/urdf/common_properties.xacro"/>
     <xacro:include filename="$(find jetbot_mirea_description)/urdf/gazebo_properties.xacro"/>
-    <link name="base_footprint"/>
+    <!-- <link name="base_footprint"/>
     <joint name="base_joint" type="fixed">
         <parent link="base_footprint"/>
         <child link="base_link"/>
         <origin xyz="0.0 0.0 ${wheel_big_radius + base_height/2}" rpy="0 0 0"/>
-    </joint>
+    </joint> -->
     <link name="base_link">
         <visual>
