Commit message: Fix lidar effrort and limits for laser filter

File: jetbot_mirea_description/urdf/jetbot_mirea_simple_gazebo_real.urdf.xacro (robot description, xacro)
@@ -125,5 +125,5 @@
         <parent link="base_link"/>
         <child link="lidar_link"/>
-        <origin xyz="0.07 0.0 ${base_height/2 + lidar_height/2}" rpy="0 0 0"/>  <!-- Поворот на -90° вокруг X -->
+        <origin xyz="0.07 0.0 ${base_height/2 + lidar_height/2}" rpy="0 0 2.3562"/>  <!-- Поворот на -90° вокруг X -->
     </joint>
     <link name="lidar_link">
